Commit message: 10.2 uppdated the URDF file with fork lift platform.

File: src/ropisim/urdf/box_bot.urdf (robot description, URDF)
Before this commit: robot sam_bot, 6 links, 5 joints
Links:
- added link platform_link, mass 1.0; collision box size=0.4 0.4 0.01; visual box size=0.4 0.4 0.01
Joints:
- added joint platform_joint: type prismatic, parent base_link, child platform_link, origin xyz=0.55 0 0.5 rpy=0 0 0, axis 0 0 1, limit lower=-0.5 upper=0.5 effort=100 velocity=0.1
